Commit message: lower masses of motors

File: catkin_ws/src/ptz_camera/models/ptz_camera/ptz_camera.urdf.xacro (robot description, xacro)
@@ -54,5 +54,5 @@
             </collision>
             <inertial>
-                <mass value="0.1"/>
+                <mass value="0.0001"/>
                 <origin xyz="0 0 0" rpy="0 0 0"/>
                 <inertia ixx="6.333e-05" ixy="0" ixz="0" iyy="6.333e-05" iyz="0" izz="0.000125"/>
@@ -83,5 +83,5 @@
             </collision>
             <inertial>
-                <mass value="0.2"/>
+                <mass value="0.00002"/>
                 <origin xyz="0 0 0" rpy="0 0 0"/>
                 <inertia ixx="0.000128" ixy="0" ixz="0" iyy="0.000128" iyz="0" izz="0.000128"/>
