Commit message: pan joint origin fix (by default pan starts at drone pov angle)

File: catkin_ws/src/hector_quadrotor_noetic/hector_models/hector_sensors_description/urdf/ptz_camera.urdf.xacro (robot description, xacro)
@@ -32,9 +32,9 @@
         <!-- Pan joint: Base to Camera (Yaw) -->
         <joint name="${name}_pan_joint" type="continuous">
-            <origin xyz="0 0 0.05" rpy="0 0 0"/>
+            <origin xyz="0 0 0.05" rpy="0 0 -1.57"/>
             <parent link="${name}_base_link"/>
             <child link="${name}_pan_link"/>
             <axis xyz="0 0 -1"/>
-            <!-- <limit lower="${-(pan_limit/2) * M_PI / 180}" upper="${(pan_limit/2) * M_PI / 180}" effort="0.001" velocity="1.0"/> -->
+            <limit lower="${-(pan_limit/2) * M_PI / 180}" upper="${(pan_limit/2) * M_PI / 180}" effort="0.001" velocity="1.0"/>
         </joint>
         <!-- Pan Link -->

Commit message: pseudozoom topics addition

File: catkin_ws/src/hector_quadrotor_noetic/hector_models/hector_sensors_description/urdf/ptz_camera.urdf.xacro (robot description, xacro)
@@ -94,6 +94,34 @@
             <child link="${name}_optical_frame"/>
         </joint>
+        <!-- Optical frame joint -->
+        <joint name="${name}_optical_joint_x2" type="fixed">
+            <origin xyz="0 0 0.05" rpy="${M_PI/2} ${-M_PI/2} 0"/>
+            <parent link="${name}_tilt_link"/>
+            <child link="${name}_optical_frame_x2"/>
+        </joint>
+        <!-- Optical frame joint -->
+        <joint name="${name}_optical_joint_x4" type="fixed">
+            <origin xyz="0 0 0.05" rpy="${M_PI/2} ${-M_PI/2} 0"/>
+            <parent link="${name}_tilt_link"/>
+            <child link="${name}_optical_frame_x4"/>
+        </joint>
         <!-- Optical Frame -->
         <link name="${name}_optical_frame">
+            <visual>
+                <geometry>
+                    <box size="0.01 0.01 0.01"/>
+                </geometry>
+            </visual>
+        </link>
+                <!-- Optical Frame -->
+        <link name="${name}_optical_frame_x2">
+            <visual>
+                <geometry>
+                    <box size="0.01 0.01 0.01"/>
+                </geometry>
+            </visual>
+        </link>
+                <!-- Optical Frame -->
+        <link name="${name}_optical_frame_x4">
             <visual>
                 <geometry>
@@ -125,4 +153,5 @@
         <gazebo>
             <plugin name="gazebo_ros_control" filename="libgazebo_ros_control.so">
+            <!-- TODO remove the uav1. this will cause problems -->
                 <robotNamespace>/uav1/${name}</robotNamespace>
                 <!-- <robotParam>/uav1/robot_description</robotParam> -->
@@ -134,5 +163,5 @@
                 <update_rate>${update_rate}</update_rate>
                 <camera>
-                <horizontal_fov>${hfov * M_PI/180.0}</horizontal_fov>
+                <horizontal_fov>1.57</horizontal_fov>
                 <image>
                     <format>${image_format}</format>
@@ -145,12 +174,62 @@
                 </clip>
                 </camera>
-                <plugin name="${name}_controller" filename="libgazebo_ros_camera.so">
+                <plugin name="camera_plugin" filename="libgazebo_ros_camera.so">
                     <cameraName>${name}</cameraName>
                     <imageTopicName>${ros_topic}</imageTopicName>
                     <cameraInfoTopicName>${cam_info_topic}</cameraInfoTopicName>
                     <frameName>${name}_optical_frame</frameName>
+                    <dynamic_parameters>true</dynamic_parameters>
+                    <horizontal_fov>1.047</horizontal_fov>
                 </plugin>
             </sensor>
         </gazebo>
+        <gazebo reference="${name}_optical_frame_x2">
+            <sensor type="camera" name="${name}_sensor_x2">
+                <update_rate>${update_rate}</update_rate>
+                <camera>
+                <horizontal_fov>0.78</horizontal_fov>
+                <image>
+                    <format>${image_format}</format>
+                    <width>${res_x}</width>
+                    <height>${res_y}</height>
+                </image>
+                <clip>
+                    <near>0.01</near>
+                    <far>100</far>
+                </clip>
+                </camera>
+                <plugin name="camera_plugin" filename="libgazebo_ros_camera.so">
+                    <cameraName>${name}_x2</cameraName>
+                    <imageTopicName>${ros_topic}_x2</imageTopicName>
+                    <cameraInfoTopicName>${cam_info_topic}</cameraInfoTopicName>
+                    <frameName>${name}_optical_frame_x2</frameName>
+                    <horizontal_fov>0.78</horizontal_fov>
+                </plugin>
+            </sensor>
+        </gazebo>
+        <gazebo reference="${name}_optical_frame_x4">
+            <sensor type="camera" name="${name}_sensor_x4">
+                <update_rate>${update_rate}</update_rate>
+                <camera>
+                <horizontal_fov>0.39</horizontal_fov>
+                <image>
+                    <format>${image_format}</format>
+                    <width>${res_x}</width>
+                    <height>${res_y}</height>
+                </image>
+                <clip>
+                    <near>0.01</near>
+                    <far>100</far>
+                </clip>
+                </camera>
+                <plugin name="camera_plugin" filename="libgazebo_ros_camera.so">
+                    <cameraName>${name}_x4</cameraName>
+                    <imageTopicName>${ros_topic}_x4</imageTopicName>
+                    <cameraInfoTopicName>${cam_info_topic}</cameraInfoTopicName>
+                    <frameName>${name}_optical_frame_x4</frameName>
+                    <horizontal_fov>0.39</horizontal_fov>
+                </plugin>
+            </sensor>
+        </gazebo>
     </xacro:macro>
 </robot>

Commit message: updated effort vals for ptz

File: catkin_ws/src/hector_quadrotor_noetic/hector_models/hector_sensors_description/urdf/ptz_camera.urdf.xacro (robot description, xacro)
@@ -36,5 +36,5 @@
             <child link="${name}_pan_link"/>
             <axis xyz="0 0 -1"/>
-            <limit lower="${-(pan_limit/2) * M_PI / 180}" upper="${(pan_limit/2) * M_PI / 180}" effort="0.001" velocity="1.0"/>
+            <limit lower="${-(pan_limit/2) * M_PI / 180}" upper="${(pan_limit/2) * M_PI / 180}" effort="0.1" velocity="1.0"/>
         </joint>
         <!-- Pan Link -->
@@ -65,5 +65,5 @@
             <child link="${name}_tilt_link"/>
             <axis xyz="1 0 0"/>
-            <limit lower="${-(tilt_limit/2) * M_PI / 180}" upper="${(tilt_limit/2) * M_PI / 180}" effort="0.001" velocity="1.0"/>
+            <limit lower="${-(tilt_limit/2) * M_PI / 180}" upper="${(tilt_limit/2) * M_PI / 180}" effort="0.1" velocity="1.0"/>
         </joint>
         <!-- Tilt Link -->

Commit message: Added roll motor

File: catkin_ws/src/hector_quadrotor_noetic/hector_models/hector_sensors_description/urdf/ptz_camera.urdf.xacro (robot description, xacro)
@@ -36,5 +36,5 @@
             <child link="${name}_pan_link"/>
             <axis xyz="0 0 -1"/>
-            <limit lower="${-(pan_limit/2) * M_PI / 180}" upper="${(pan_limit/2) * M_PI / 180}" effort="0.1" velocity="1.0"/>
+            <limit lower="${-(pan_limit/2) * M_PI / 180}" upper="${(pan_limit/2) * M_PI / 180}" effort="1.0" velocity="1.0"/>
         </joint>
         <!-- Pan Link -->
@@ -65,8 +65,37 @@
             <child link="${name}_tilt_link"/>
             <axis xyz="1 0 0"/>
-            <limit lower="${-(tilt_limit/2) * M_PI / 180}" upper="${(tilt_limit/2) * M_PI / 180}" effort="0.1" velocity="1.0"/>
+            <limit lower="${-(tilt_limit/2) * M_PI / 180}" upper="${(tilt_limit/2) * M_PI / 180}" effort="1000.0" velocity="1.0"/>
         </joint>
         <!-- Tilt Link -->
         <link name="${name}_tilt_link">
+            <visual>
+                <geometry>
+                    <sphere radius="0.04"/>
+                </geometry>
+                <material name="gray">
+                    <color rgba="0.7 0.7 0.7 1.0"/>
+                </material>
+            </visual>
+            <collision>
+                <geometry>
+                    <sphere radius="0.04"/>
+                </geometry>
+            </collision>
+            <inertial>
+                <mass value="0.2"/>
+                <origin xyz="0 0 0" rpy="0 0 0"/>
+                <inertia ixx="0.000128" ixy="0" ixz="0" iyy="0.000128" iyz="0" izz="0.000128"/>
+            </inertial>
+        </link>
+        <!-- Roll joint: roll Link to Camera Link (Roll) -->
+        <joint name="${name}_roll_joint" type="revolute">
+            <origin xyz="0 0 0.005" rpy="0 0 0"/>
+            <parent link="${name}_tilt_link"/>
+            <child link="${name}_roll_link"/>
+            <axis xyz="0 1 0"/>
+            <limit lower="${-(tilt_limit/2) * M_PI / s180}" upper="${(tilt_limit/2) * M_PI / 180}" effort="1000.0" velocity="1.0"/>
+        </joint>
+        <!-- Tilt Link -->
+        <link name="${name}_roll_link">
             <visual>
                 <geometry>
@@ -91,5 +120,5 @@
         <joint name="${name}_optical_joint" type="fixed">
             <origin xyz="0 0 0.05" rpy="${M_PI/2} ${-M_PI/2} 0"/>
-            <parent link="${name}_tilt_link"/>
+            <parent link="${name}_roll_link"/>
             <child link="${name}_optical_frame"/>
         </joint>
@@ -97,5 +126,5 @@
         <joint name="${name}_optical_joint_x2" type="fixed">
             <origin xyz="0 0 0.05" rpy="${M_PI/2} ${-M_PI/2} 0"/>
-            <parent link="${name}_tilt_link"/>
+            <parent link="${name}_roll_link"/>
             <child link="${name}_optical_frame_x2"/>
         </joint>
@@ -103,5 +132,5 @@
         <joint name="${name}_optical_joint_x4" type="fixed">
             <origin xyz="0 0 0.05" rpy="${M_PI/2} ${-M_PI/2} 0"/>
-            <parent link="${name}_tilt_link"/>
+            <parent link="${name}_roll_link"/>
             <child link="${name}_optical_frame_x4"/>
         </joint>
@@ -147,4 +176,14 @@
             </joint>
             <actuator name="${name}_tilt_joint_motor">
+                <hardwareInterface>hardware_interface/PositionJointInterface</hardwareInterface>
+                <mechanicalReduction>1</mechanicalReduction>
+            </actuator>
+        </transmission>
+        <transmission name="${name}_roll_joint_trans">
+            <type>transmission_interface/SimpleTransmission</type>
+            <joint name="${name}_roll_joint">
+                <hardwareInterface>hardware_interface/PositionJointInterface</hardwareInterface>
+            </joint>
+            <actuator name="${name}_roll_joint_motor">
                 <hardwareInterface>hardware_interface/PositionJointInterface</hardwareInterface>
                 <mechanicalReduction>1</mechanicalReduction>

Commit message: ptz changes - should be working

File: catkin_ws/src/hector_quadrotor_noetic/hector_models/hector_sensors_description/urdf/ptz_camera.urdf.xacro (robot description, xacro)
@@ -25,5 +25,5 @@
             </collision>
             <inertial>
-                <mass value="0.5"/>
+                <mass value="0.05"/>
                 <origin xyz="0 0 0" rpy="0 0 0"/>
                 <inertia ixx="0.000833" ixy="0" ixz="0" iyy="0.000833" iyz="0" izz="0.000833"/>
@@ -54,5 +54,5 @@
             </collision>
             <inertial>
-                <mass value="0.1"/>
+                <mass value="0.0001"/>
                 <origin xyz="0 0 0" rpy="0 0 0"/>
                 <inertia ixx="6.333e-05" ixy="0" ixz="0" iyy="6.333e-05" iyz="0" izz="0.000125"/>
@@ -60,10 +60,11 @@
         </link>
         <!-- Tilt joint: Pan Link to Camera Link (Pitch) -->
-        <joint name="${name}_tilt_joint" type="revolute">
+        <joint name="${name}_tilt_joint" type="continuous">
             <origin xyz="0 0 0.005" rpy="0 0 0"/>
             <parent link="${name}_pan_link"/>
             <child link="${name}_tilt_link"/>
             <axis xyz="1 0 0"/>
-            <limit lower="${-(tilt_limit/2) * M_PI / 180}" upper="${(tilt_limit/2) * M_PI / 180}" effort="1000.0" velocity="1.0"/>
+            <!-- <limit lower="${-(tilt_limit/2) * M_PI / 180}" upper="${(tilt_limit/2) * M_PI / 180}" effort="10.0" velocity="10.0"/> -->
+            <limit lower="${-(pan_limit/2) * M_PI / 180}" upper="${(pan_limit/2) * M_PI / 180}" effort="100.0" velocity="100.0"/>
         </joint>
         <!-- Tilt Link -->
@@ -83,5 +84,5 @@
             </collision>
             <inertial>
-                <mass value="0.2"/>
+                <mass value="0.0002"/>
                 <origin xyz="0 0 0" rpy="0 0 0"/>
                 <inertia ixx="0.000128" ixy="0" ixz="0" iyy="0.000128" iyz="0" izz="0.000128"/>
@@ -89,10 +90,10 @@
         </link>
         <!-- Roll joint: roll Link to Camera Link (Roll) -->
-        <joint name="${name}_roll_joint" type="revolute">
-            <origin xyz="0 0 0.005" rpy="0 0 0"/>
+        <joint name="${name}_roll_joint" type="continuous">
+            <origin xyz="0 0.06 0.01" rpy="0 0 0"/>
             <parent link="${name}_tilt_link"/>
             <child link="${name}_roll_link"/>
             <axis xyz="0 1 0"/>
-            <limit lower="${-(tilt_limit/2) * M_PI / s180}" upper="${(tilt_limit/2) * M_PI / 180}" effort="1000.0" velocity="1.0"/>
+            <limit lower="${-(pan_limit/2) * M_PI / 180}" upper="${(pan_limit/2) * M_PI / 180}" effort="100.0" velocity="100.0"/>
         </joint>
         <!-- Tilt Link -->
@@ -112,5 +113,5 @@
             </collision>
             <inertial>
-                <mass value="0.2"/>
+                <mass value="0.0002"/>
                 <origin xyz="0 0 0" rpy="0 0 0"/>
                 <inertia ixx="0.000128" ixy="0" ixz="0" iyy="0.000128" iyz="0" izz="0.000128"/>

Commit message: updated the stabilization

File: catkin_ws/src/hector_quadrotor_noetic/hector_models/hector_sensors_description/urdf/ptz_camera.urdf.xacro (robot description, xacro)
@@ -25,5 +25,5 @@
             </collision>
             <inertial>
-                <mass value="0.05"/>
+                <mass value="0.0005"/>
                 <origin xyz="0 0 0" rpy="0 0 0"/>
                 <inertia ixx="0.000833" ixy="0" ixz="0" iyy="0.000833" iyz="0" izz="0.000833"/>
@@ -36,5 +36,5 @@
             <child link="${name}_pan_link"/>
             <axis xyz="0 0 -1"/>
-            <limit lower="${-(pan_limit/2) * M_PI / 180}" upper="${(pan_limit/2) * M_PI / 180}" effort="1.0" velocity="1.0"/>
+            <limit lower="${-(pan_limit/2) * M_PI / 180}" upper="${(pan_limit/2) * M_PI / 180}" effort="10.0" velocity="1.0"/>
         </joint>
         <!-- Pan Link -->
@@ -66,5 +66,5 @@
             <axis xyz="1 0 0"/>
             <!-- <limit lower="${-(tilt_limit/2) * M_PI / 180}" upper="${(tilt_limit/2) * M_PI / 180}" effort="10.0" velocity="10.0"/> -->
-            <limit lower="${-(pan_limit/2) * M_PI / 180}" upper="${(pan_limit/2) * M_PI / 180}" effort="100.0" velocity="100.0"/>
+            <limit lower="${-(pan_limit/2) * M_PI / 180}" upper="${(pan_limit/2) * M_PI / 180}" effort="10000.0" velocity="100.0"/>
         </joint>
         <!-- Tilt Link -->
@@ -84,5 +84,5 @@
             </collision>
             <inertial>
-                <mass value="0.0002"/>
+                <mass value="0.0001"/>
                 <origin xyz="0 0 0" rpy="0 0 0"/>
                 <inertia ixx="0.000128" ixy="0" ixz="0" iyy="0.000128" iyz="0" izz="0.000128"/>
@@ -95,5 +95,5 @@
             <child link="${name}_roll_link"/>
             <axis xyz="0 1 0"/>
-            <limit lower="${-(pan_limit/2) * M_PI / 180}" upper="${(pan_limit/2) * M_PI / 180}" effort="100.0" velocity="100.0"/>
+            <limit lower="${-(pan_limit/2) * M_PI / 180}" upper="${(pan_limit/2) * M_PI / 180}" effort="10000.0" velocity="100.0"/>
         </joint>
         <!-- Tilt Link -->
