Commit message: vroom?

File: catkin_ws/src/hector_quadrotor_noetic/hector_models/hector_sensors_description/urdf/ptz_camera.urdf.xacro (robot description, xacro)
@@ -36,5 +36,5 @@
             <child link="${name}_pan_link"/>
             <axis xyz="0 0 -1"/>
-            <limit lower="${-(pan_limit/2) * M_PI / 180}" upper="${(pan_limit/2) * M_PI / 180}" effort="10.0" velocity="1.0"/>
+            <limit lower="${-(pan_limit/2) * M_PI / 180}" upper="${(pan_limit/2) * M_PI / 180}" effort="1000.0" velocity="1.0"/>
         </joint>
         <!-- Pan Link -->
@@ -60,11 +60,11 @@
         </link>
         <!-- Tilt joint: Pan Link to Camera Link (Pitch) -->
-        <joint name="${name}_tilt_joint" type="continuous">
+        <joint name="${name}_tilt_joint" type="revolute">
             <origin xyz="0 0 0.005" rpy="0 0 0"/>
             <parent link="${name}_pan_link"/>
             <child link="${name}_tilt_link"/>
             <axis xyz="1 0 0"/>
-            <!-- <limit lower="${-(tilt_limit/2) * M_PI / 180}" upper="${(tilt_limit/2) * M_PI / 180}" effort="10.0" velocity="10.0"/> -->
-            <limit lower="${-(pan_limit/2) * M_PI / 180}" upper="${(pan_limit/2) * M_PI / 180}" effort="10000.0" velocity="100.0"/>
+            <limit lower="${-(tilt_limit/2) * M_PI / 180}" upper="${(tilt_limit/2) * M_PI / 180}" effort="10000.0" velocity="100.0"/>
+            <!-- <limit lower="${-(pan_limit/2) * M_PI / 180}" upper="${(pan_limit/2) * M_PI / 180}" effort="10000.0" velocity="100.0"/> -->
         </joint>
         <!-- Tilt Link -->
@@ -90,10 +90,11 @@
         </link>
         <!-- Roll joint: roll Link to Camera Link (Roll) -->
-        <joint name="${name}_roll_joint" type="continuous">
+        <joint name="${name}_roll_joint" type="revolute">
             <origin xyz="0 0.06 0.01" rpy="0 0 0"/>
             <parent link="${name}_tilt_link"/>
             <child link="${name}_roll_link"/>
             <axis xyz="0 1 0"/>
-            <limit lower="${-(pan_limit/2) * M_PI / 180}" upper="${(pan_limit/2) * M_PI / 180}" effort="10000.0" velocity="100.0"/>
+            <limit lower="${-(tilt_limit/2) * M_PI / 180}" upper="${(tilt_limit/2) * M_PI / 180}" effort="10000.0" velocity="100.0"/>
+            <!-- <limit lower="${-(pan_limit/2) * M_PI / 180}" upper="${(pan_limit/2) * M_PI / 180}" effort="10000.0" velocity="100.0"/> -->
         </joint>
         <!-- Tilt Link -->

File: catkin_ws/src/multi_robot_scenario/xacro/camera/camera.xacro (robot description, xacro)
@@ -39,6 +39,8 @@
         <horizontal_fov>1.92</horizontal_fov>
         <image>
-          <width>512</width>
-          <height>256</height>
+          <!-- <width>512</width>
+          <height>256</height> -->
+          <width>160</width>
+          <height>160</height>
           <format>R8G8B8</format>
         </image>

File: catkin_ws/src/multi_robot_scenario/xacro/cylinder_robot/cylinder_robot_chassis.xacro (robot description, xacro)
@@ -20,14 +20,10 @@
     </visual>
     <collision>
-      <!-- <origin xyz="-0.045 0 0.148" rpy="0 0 0"/> -->
-      <!-- <origin xyz="-0.045 0 0.148" rpy="0 0 0"/> -->
-      <origin xyz="-0.045 0 0.14" rpy="0 0 0"/>
-      <!-- <origin xyz="-0 0 0" rpy="0 0 0"/> -->
+      <origin xyz="-0.045 0 0.148" rpy="0 0 0"/>
       <geometry>
         <mesh filename="${meshes}/chassis.stl"/>
       </geometry>
     </collision>
-    <!-- <xacro:box_inertial x="0.36" y="0.26"  z="0.18" mass="9.0" /> -->
-    <xacro:cylinder_inertial radius="0.25" length="0.2" mass="18.0" />
+    <xacro:box_inertial x="0.36" y="0.26"  z="0.18" mass="9.0" />
   </link>
   <joint name="${parent}_box_joint" type="fixed">
@@ -40,5 +36,5 @@
       <origin xyz="-0.045 0 0.14" rpy="0 0 0"/>
       <geometry>
-          <cylinder length="0.05" radius="0.25"/>
+          <cylinder length="0.005" radius="0.25"/>
         </geometry>
       <material name="ChassisRed">
@@ -47,11 +43,10 @@
     </visual>
     <collision>
-      <origin xyz="-0.045 0 0.1" rpy="0 0 0"/>
+      <origin xyz="-0.045 0 0.14" rpy="0 0 0"/>
       <geometry>
           <cylinder length="0.005" radius="0.25"/>
         </geometry>
     </collision>
-    <!-- <xacro:box_inertial x="0.36" y="0.26"  z="0.18" mass="9.0" /> -->
-    <xacro:cylinder_inertial radius="0.25" length="0.005" mass="1.0" />
+    <xacro:box_inertial x="0.36" y="0.26"  z="0.18" mass="9.0" />
   </link>
   <!-- Contact Sensor -->
@@ -87,11 +82,10 @@
     </visual>
     <collision>
-    <origin xyz="0 0 -0.1" rpy="0 0 0"/>
+    <origin xyz="0.0 0 0.0" rpy="0 0 0"/>
       <geometry>
         <mesh filename="${meshes}/top.stl"/>
       </geometry>
     </collision>
-    <!-- <xacro:box_inertial x="0.445" y="0.38"  z="0.01" mass="1.0" /> -->
-    <xacro:cylinder_inertial radius="0.2" length="0.01" mass="0.1" />
+    <xacro:box_inertial x="0.445" y="0.38"  z="0.01" mass="1.0" />
   </link>
   <gazebo reference="top">

File: catkin_ws/src/multi_robot_scenario/xacro/p3dx/pioneer3dx.xacro (robot description, xacro)
@@ -6,7 +6,9 @@
   <xacro:include filename="$(find multi_robot_scenario)/xacro/p3dx/pioneer3dx_body.xacro"/>
   <xacro:pioneer3dx_body name="chassis" parent="base_link" meshes="package://gazebo_plugins/test/multi_robot_scenario/meshes/p3dx"/>
+  <!-- <xacro:include filename="$(find multi_robot_scenario)/xacro/cylinder_robot/cylinder_robot_body.xacro"/>
+  <xacro:pioneer3dx_body name="chassis" parent="base_link" meshes="package://gazebo_plugins/test/multi_robot_scenario/meshes/p3dx"/> -->
   <!-- Laser -->
-  <xacro:include filename="$(find multi_robot_scenario)/xacro/laser/hokuyo.xacro"/>
-  <xacro:laser name="front_laser" parent="chassis" xyz="0.125 0 0.25" rpy="0 0 0" meshes="package://gazebo_plugins/test/multi_robot_scenario/meshes/laser"/>
+  <!-- <xacro:include filename="$(find multi_robot_scenario)/xacro/laser/hokuyo.xacro"/>
+  <xacro:laser name="front_laser" parent="chassis" xyz="0.125 0 0.25" rpy="0 0 0" meshes="package://gazebo_plugins/test/multi_robot_scenario/meshes/laser"/> -->
   <!-- GPU Laser
   <xacro:include filename="$(find multi_robot_scenario)/xacro/laser/hokuyo_gpu.xacro"/>
@@ -18,7 +20,7 @@
   <xacro:camD name="cameraD" parent="chassis" xyz="0.025 0 0.32" rpy="0 0 0" /> -->
   <!-- Velodyne -->
-  <xacro:include filename="$(find velodyne_description)/urdf/VLP-16.urdf.xacro"/>
+  <!-- <xacro:include filename="$(find velodyne_description)/urdf/VLP-16.urdf.xacro"/>
   <xacro:VLP-16 parent="base_link" name="velodyne" topic="/velodyne_points" hz="10" samples="360" gpu="false" min_angle="-1.57" max_angle="1.57" min_range="0.1">
     <origin xyz="0.125 0 0.25" rpy="0 0 0" />
-  </xacro:VLP-16>
+  </xacro:VLP-16> -->
 </robot>

File: catkin_ws/src/multi_robot_scenario/xacro/p3dx/pioneer3dx_body.xacro (robot description, xacro)
@@ -14,15 +14,16 @@
     <xacro:pioneer_chassis name="${name}" parent="base_link" xyz="0 0 0" rpy="0 0 0"  meshes="${meshes}"/>
     <!-- Front Sonar -->
-    <xacro:pioneer_sonar name="sonar" parent="${name}" xyz="0.109 0 0.209" rpy="0 0 0"  meshes="${meshes}"/>
+    <!-- <xacro:pioneer_sonar name="sonar" parent="${name}" xyz="0.109 0 0.209" rpy="0 0 0"  meshes="${meshes}"/> -->
     <!-- Akku0 -->
-    <xacro:battery_block name="battery0" parent="${name}" x="-0.14" y="0.00"  z="0.13" mass="2.5" />
+    <!-- <xacro:battery_block name="battery0" parent="${name}" x="-0.14" y="0.00"  z="0.13" mass="2.5" /> -->
     <!-- Wheels -->
-    <xacro:pioneer_wheel side="right" parent="${name}"  xyz="0  0.15 0.09" rpy="0 0 0" radius="0.09" meshes="${meshes}"/>
+    <!-- <xacro:pioneer_wheel side="right" parent="${name}"  xyz="0  0.15 0.09" rpy="0 0 0" radius="0.09" meshes="${meshes}"/>
     <xacro:pioneer_wheel side="left"  parent="${name}"  xyz="0 -0.15 0.09" rpy="0 0 0" radius="0.09" meshes="${meshes}"/>
-    <xacro:pioneer_swivel parent="${name}"  xyz="-0.185 0 0.055" rpy="0 0 0" meshes="${meshes}"/>
+    <xacro:pioneer_swivel parent="${name}"  xyz="-0.185 0 0.055" rpy="0 0 0" meshes="${meshes}"/> -->
     <!-- Motor plugin -->
-    <xacro:pioneer3dx_diff_drive />
+    <!-- <xacro:pioneer3dx_diff_drive />  -->
     <!-- Joints plugin -->
-    <xacro:pioneer3dx_joints_state_publisher />
+    <!-- <xacro:pioneer3dx_joints_state_publisher /> -->
+    <xacro:pioneer3dx_pose />
   </xacro:macro>
 </robot>

File: catkin_ws/src/multi_robot_scenario/xacro/p3dx/pioneer3dx_plugins.xacro (robot description, xacro)
@@ -8,4 +8,11 @@
           <updateRate>50.0</updateRate>
           <alwaysOn>true</alwaysOn>
+        </plugin>
+    </gazebo>
+  </xacro:macro>
+  <xacro:macro name="pioneer3dx_pose">
+    <gazebo>
+        <plugin name="robot_pose_publisher" filename="librobot_pose_publisher.so">
+	        <updateRate>100</updateRate>
         </plugin>
     </gazebo>
@@ -30,5 +37,5 @@
             <odometrySource>world</odometrySource>
             <robotBaseFrame>base_link</robotBaseFrame>
-	    <updateRate>50</updateRate>
+	    <updateRate>100</updateRate>
         </plugin>
     </gazebo>

File: catkin_ws/src/velodyne_simulator/velodyne_description/urdf/VLP-16.urdf.xacro (robot description, xacro)
@@ -49,4 +49,5 @@
           <mesh filename="package://velodyne_description/meshes/VLP16_scan.dae" />
         </geometry>
+          <plugin name="gazebo_ros_laser_controller" filename="libga
       </visual> -->
     </link>
