Commit message: splitting into lidar, cam and default

File: catkin_ws/src/multi_robot_scenario/xacro/p3dx/pioneer3dx_body_fast.xacro (robot description, xacro)
@@ -8,5 +8,5 @@
   <xacro:include filename="pioneer3dx_sonar.xacro"/>
   <xacro:include filename="pioneer3dx_plugins.xacro"/>
-  <xacro:macro name="pioneer3dx_body" params="name parent meshes">
+  <xacro:macro name="pioneer3dx_body_fast" params="name parent meshes">
     <!-- base_link -->
     <link name="${parent}"/>
@@ -16,13 +16,13 @@
     <!-- <xacro:pioneer_sonar name="sonar" parent="${name}" xyz="0.109 0 0.209" rpy="0 0 0"  meshes="${meshes}"/> -->
     <!-- Akku0 -->
-    <xacro:battery_block name="battery0" parent="${name}" x="-0.14" y="0.00"  z="0.13" mass="2.5" />
+    <!-- <xacro:battery_block name="battery0" parent="${name}" x="-0.14" y="0.00"  z="0.13" mass="2.5" /> -->
     <!-- Wheels -->
-    <xacro:pioneer_wheel side="right" parent="${name}"  xyz="0  0.15 0.09" rpy="0 0 0" radius="0.09" meshes="${meshes}"/>
+    <!-- <xacro:pioneer_wheel side="right" parent="${name}"  xyz="0  0.15 0.09" rpy="0 0 0" radius="0.09" meshes="${meshes}"/>
     <xacro:pioneer_wheel side="left"  parent="${name}"  xyz="0 -0.15 0.09" rpy="0 0 0" radius="0.09" meshes="${meshes}"/>
-    <xacro:pioneer_swivel parent="${name}"  xyz="-0.185 0 0.055" rpy="0 0 0" meshes="${meshes}"/>
+    <xacro:pioneer_swivel parent="${name}"  xyz="-0.185 0 0.055" rpy="0 0 0" meshes="${meshes}"/> -->
     <!-- Motor plugin -->
-    <xacro:pioneer3dx_diff_drive />
+    <!-- <xacro:pioneer3dx_diff_drive />  -->
     <!-- Joints plugin -->
-    <xacro:pioneer3dx_joints_state_publisher />
+    <!-- <xacro:pioneer3dx_joints_state_publisher /> -->
     <xacro:pioneer3dx_pose />
   </xacro:macro>
